File: SuperLoader.kicad_pcb (KiCad board)
At the start: 2 copper layers, 82 x 51 mm, 38 parts, among them J1 EAR in, J2 9V DC in, J3 9V DC(out), J4 Out, U1 LM324, U2 NE555P

Commit message: Added copper logo and fixed symbol
Parts:
- removed the REF** at (58.5, 50.6)
- added G200: LOGO, ZXLibrary:ZXInfo_kicad_logo, F.Cu at (76.9, 29.5)
- added REF**: Logo, ZXLibrary:Logo, F.Cu at (75.0, 40.6)
